File: swerveDriveTrain/swerveDriveTrain.kicad_pcb (KiCad board)
At the start: 4 copper layers, 82.5 x 125.6 mm, 29 parts, among them IC1 TCAN3414DR, J1 RJ45, J2 Screw_Terminal_01x02, J3 Conn_01x06_Pin, J4 S6B-PH-K-S_LF__SN_, U1 G218v17, U2 Teensy4.0, U3 G218v17

Commit message: finalize pcb
Parts:
- added C10: 0.1uF, Capacitor_SMD:C_0805_2012Metric_Pad1.18x1.45mm_HandSolder, F.Cu at (240.7, 79.5)
- added C5: 22uF, Capacitor_SMD:C_0805_2012Metric_Pad1.18x1.45mm_HandSolder, F.Cu at (244.5, 65.9)
- added C6: 22uF, Capacitor_SMD:C_0805_2012Metric_Pad1.18x1.45mm_HandSolder, F.Cu at (244.5, 68.2)
- added C7: 0.1uF, Capacitor_SMD:C_0805_2012Metric_Pad1.18x1.45mm_HandSolder, F.Cu at (238.7, 76.5)
- added C8: 10uF, Capacitor_SMD:C_0805_2012Metric_Pad1.18x1.45mm_HandSolder, F.Cu at (240.7, 84.0)
- added C9: 10uF, Capacitor_SMD:C_0805_2012Metric_Pad1.18x1.45mm_HandSolder, F.Cu at (240.7, 81.8)
- added L3: 3.3uH, Inductor_SMD:L_Abracon_ASPI-0630LR, F.Cu at (237.9, 69.9)
- added R12: 10K, Resistor_SMD:R_0805_2012Metric_Pad1.20x1.40mm_HandSolder, F.Cu at (247.9, 73.6)
- added R13: 54.9K, Resistor_SMD:R_0805_2012Metric_Pad1.20x1.40mm_HandSolder, F.Cu at (244.5, 70.7)
- added U4: TPS565208, Package_TO_SOT_SMD:SOT-23-6, F.Cu at (242.9, 75.5)
- moved L2 12.3 mm to (219.1, 68.0)
- moved TP11 9.43 mm to (242.0, 116.0)
- moved TP12 9.42 mm to (242.0, 124.8)
- moved TP13 9.42 mm to (242.0, 120.5)
- moved R3 2.20 mm to (200.4, 32.2)
- moved R8 2.17 mm to (193.1, 32.0)
- moved R1 1.70 mm to (213.2, 32.3)
- moved R2 1.36 mm to (206.4, 32.2)
- moved D4 0.50 mm to (193.1, 25.9), turned to -90 degrees
- moved D3 0.23 mm to (200.4, 26.0), turned to -90 degrees
- moved C4 0.20 mm to (198.1, 142.5)
- moved D2 0.08 mm to (206.4, 26.1), turned to -90 degrees
- turned D1 to -90 degrees
Routing:
- net +12V: track 1.49 -> 205.7 mm, vias 0 -> 2
- net +5V: track 131.8 -> 216.4 mm, vias 1 -> 5
- net LED1: track 0.00 -> 35.1 mm
- net LED2: track 0.00 -> 33.0 mm
- net GND: track 14.4 -> 29.8 mm, vias 8 -> 71
- net Net-(U4-VBST): track 0.00 -> 11.1 mm, vias 0 -> 2
- net Net-(U4-VFB): track 0.00 -> 8.34 mm
- net Net-(U4-SW): track 0.00 -> 5.92 mm
- net Net-(D3-A): track 0.00 -> 4.18 mm
- net Net-(D2-A): track 0.00 -> 4.08 mm
- net Net-(D1-A): track 0.00 -> 4.07 mm
- net Net-(D4-A): track 0.00 -> 4.03 mm
- net M1B: track 64.1 -> 61.5 mm
- net M1A: track 69.1 -> 67.9 mm
- net CAN3v3: track 131.1 -> 132.0 mm
Other:
- board text removed: "RGB"
