File: swerveDriveTrain/swerveDriveTrain.kicad_sch (KiCad schematic)
At the start: 39 parts, among them IC1 TCAN3414DR, J1 RJ45, J2 Screw_Terminal_01x02, J3 Conn_01x06_Pin, J4 S6B-PH-K-S_LF__SN_, U2 Teensy4.0

Commit message: new outline
Other:
- moved on the sheet: C4, IC1
Changed lines of the file:
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@@
 	)
 	(junction
-		(at 102.87 173.99)
+		(at 191.77 86.36)
 		(diameter 0)
 		(color 0 0 0 0)
@@
 	(wire
 		(pts
-			(xy 96.52 173.99) (xy 102.87 173.99)
+			(xy 185.42 86.36) (xy 191.77 86.36)
 		)
 		(stroke
@@
 	(wire
 		(pts
-			(xy 157.48 175.26) (xy 148.59 175.26)
+			(xy 246.38 87.63) (xy 237.49 87.63)
 		)
 		(stroke
@@
 	(wire
 		(pts
-			(xy 106.68 177.8) (xy 115.57 177.8)
+			(xy 195.58 90.17) (xy 204.47 90.17)
 		)
 		(stroke
@@
 	(wire
 		(pts
-			(xy 106.68 180.34) (xy 115.57 180.34)
+			(xy 195.58 92.71) (xy 204.47 92.71)
 		)
 		(stroke
@@
 	(wire
 		(pts
-			(xy 106.68 173.99) (xy 106.68 177.8)
+			(xy 195.58 86.36) (xy 195.58 90.17)
 		)
 		(stroke
@@
 	(wire
 		(pts
-			(xy 102.87 181.61) (xy 106.68 181.61)
+			(xy 191.77 93.98) (xy 195.58 93.98)
 		)
 		(stroke
@@
 	(wire
 		(pts
-			(xy 102.87 173.99) (xy 106.68 173.99)
+			(xy 191.77 86.36) (xy 195.58 86.36)
 		)
 		(stroke
@@
 	(wire
 		(pts
-			(xy 106.68 181.61) (xy 106.68 180.34)
+			(xy 195.58 93.98) (xy 195.58 92.71)
 		)
 		(stroke
@@
 	(text_box "CAN transiever will pull <250mA if using 3414 if we need any more 3.3 we should switch this over to a real reg\n"
 		(exclude_from_sim no)
-		(at 86.36 158.75 0)
+		(at 175.26 71.12 0)
 		(size 27.94 12.7)
 		(stroke
@@
 	(global_label "CAN3v3"
 		(shape input)
-		(at 102.87 181.61 180)
+		(at 191.77 93.98 180)
 		(fields_autoplaced yes)
 		(effects
@@
 		)
 		(property "Intersheetrefs" "${INTERSHEET_REFS}"
-			(at 92.8091 181.61 0)
+			(at 181.7091 93.98 0)
 			(effects
 				(font
@@
 	(global_label "CTX"
 		(shape input)
-		(at 115.57 175.26 180)
+		(at 204.47 87.63 180)
 		(fields_autoplaced yes)
 		(effects
@@
 		)
 		(property "Intersheetrefs" "${INTERSHEET_REFS}"
-			(at 109.1377 175.26 0)
+			(at 198.0377 87.63 0)
 			(effects
 				(font
@@
 	(global_label "CRX"
 		(shape input)
-		(at 115.57 182.88 180)
+		(at 204.47 95.25 180)
 		(fields_autoplaced yes)
 		(effects
@@
 		)
 		(property "Intersheetrefs" "${INTERSHEET_REFS}"
-			(at 108.8353 182.88 0)
+			(at 197.7353 95.25 0)
 			(effects
 				(font
@@
 	(global_label "CANP"
 		(shape input)
-		(at 148.59 177.8 0)
+		(at 237.49 90.17 0)
 		(fields_autoplaced yes)
 		(effects
@@
 		)
 		(property "Intersheetrefs" "${INTERSHEET_REFS}"
-			(at 155.8801 177.8 0)
+			(at 244.7801 90.17 0)
 			(effects
 				(font
@@
 	(global_label "CANN"
 		(shape input)
-		(at 148.59 180.34 0)
+		(at 237.49 92.71 0)
 		(fields_autoplaced yes)
 		(effects
@@
 		)
 		(property "Intersheetrefs" "${INTERSHEET_REFS}"
-			(at 155.9406 180.34 0)
+			(at 244.8406 92.71 0)
 			(effects
 				(font
@@
 	(symbol
 		(lib_id "power:GND")
-		(at 157.48 175.26 0)
+		(at 246.38 87.63 0)
 		(unit 1)
 		(exclude_from_sim no)
@@
 		(fields_autoplaced yes)
 		(property "Reference" "#PWR042"
-			(at 157.48 181.61 0)
+			(at 246.38 93.98 0)
 			(effects
 				(font
@@
 		)
 		(property "Value" "GND"
-			(at 160.02 176.5299 0)
+			(at 248.92 88.8999 0)
 			(effects
 				(font
@@
 		)
 		(property "Footprint" ""
-			(at 157.48 175.26 0)
+			(at 246.38 87.63 0)
 			(effects
 				(font
@@
 		)
 		(property "Datasheet" ""
-			(at 157.48 175.26 0)
+			(at 246.38 87.63 0)
 			(effects
 				(font
@@
 		)
 		(property "Description" "Power symbol creates a global label with name \"GND\" , ground"
-			(at 157.48 175.26 0)
+			(at 246.38 87.63 0)
 			(effects
 				(font
@@
 	(symbol
 		(lib_id "TCAN3414DR:TCAN3414DR")
-		(at 115.57 175.26 0)
+		(at 204.47 87.63 0)
 		(unit 1)
 		(exclude_from_sim no)
@@
 		(fields_autoplaced yes)
 		(property "Reference" "IC1"
-			(at 132.08 167.64 0)
+			(at 220.98 80.01 0)
 			(effects
 				(font
@@
 		)
 		(property "Value" "TCAN3414DR"
-			(at 132.08 170.18 0)
+			(at 220.98 82.55 0)
 			(effects
 				(font
@@
 		)
 		(property "Footprint" "footprints:SOIC127P600X175-8N"
-			(at 144.78 270.18 0)
+			(at 233.68 182.55 0)
 			(effects
 				(font
@@
 		)
 		(property "Datasheet" "https://www.ti.com/lit/ds/symlink/tcan3414.pdf?ts=1713723144569&ref_url=https%253A%252F%252Fwww.mouser.ch%252F"
-			(at 144.78 370.18 0)
+			(at 233.68 282.55 0)
 			(effects
 				(font
@@
 		)
 		(property "Description" "3.3-V CAN FD transceiver with shut-down and standby mode"
-			(at 115.57 175.26 0)
+			(at 204.47 87.63 0)
 			(effects
 				(font
@@
 		)
 		(property "Height" "1.75"
-			(at 144.78 570.18 0)
+			(at 233.68 482.55 0)
 			(effects
 				(font
@@
 		)
 		(property "Mouser Part Number" "595-TCAN3414DR"
-			(at 144.78 670.18 0)
+			(at 233.68 582.55 0)
 			(effects
 				(font
@@
 		)
 		(property "Mouser Price/Stock" "https://www.mouser.co.uk/ProductDetail/Texas-Instruments/TCAN3414DR?qs=mELouGlnn3egF2AojRJddw%3D%3D"
-			(at 144.78 770.18 0)
+			(at 233.68 682.55 0)
 			(effects
 				(font
@@
 		)
 		(property "Manufacturer_Name" "Texas Instruments"
-			(at 144.78 870.18 0)
+			(at 233.68 782.55 0)
 			(effects
 				(font
@@
 		)
 		(property "Manufacturer_Part_Number" "TCAN3414DR"
-			(at 144.78 970.18 0)
+			(at 233.68 882.55 0)
 			(effects
 				(font
@@
 	(symbol
 		(lib_id "power:GND")
-		(at 148.59 182.88 0)
+		(at 237.49 95.25 0)
 		(unit 1)
 		(exclude_from_sim no)
@@
 		(fields_autoplaced yes)
 		(property "Reference" "#PWR044"
-			(at 148.59 189.23 0)
+			(at 237.49 101.6 0)
 			(effects
 				(font
@@
 		)
 		(property "Value" "GND"
-			(at 151.13 184.1499 0)
+			(at 240.03 96.5199 0)
 			(effects
 				(font
@@
 		)
 		(property "Footprint" ""
-			(at 148.59 182.88 0)
+			(at 237.49 95.25 0)
 			(effects
 				(font
@@
 		)
 		(property "Datasheet" ""
-			(at 148.59 182.88 0)
+			(at 237.49 95.25 0)
 			(effects
 				(font
@@
 		)
 		(property "Description" "Power symbol creates a global label with name \"GND\" , ground"
-			(at 148.59 182.88 0)
+			(at 237.49 95.25 0)
 			(effects
 				(font
@@
 	(symbol
 		(lib_id "power:GND")
-		(at 96.52 173.99 0)
+		(at 185.42 86.36 0)
 		(unit 1)
 		(exclude_from_sim no)
@@
 		(dnp no)
 		(property "Reference" "#PWR041"
-			(at 96.52 180.34 0)
+			(at 185.42 92.71 0)
 			(effects
 				(font
@@
 		)
 		(property "Value" "GND"
-			(at 96.52 177.8 0)
+			(at 185.42 90.17 0)
 			(effects
 				(font
@@
 		)
 		(property "Footprint" ""
-			(at 96.52 173.99 0)
+			(at 185.42 86.36 0)
 			(effects
 				(font
@@
 		)
 		(property "Datasheet" ""
-			(at 96.52 173.99 0)
+			(at 185.42 86.36 0)
 			(effects
 				(font
@@
 		)
 		(property "Description" "Power symbol creates a global label with name \"GND\" , ground"
-			(at 96.52 173.99 0)
+			(at 185.42 86.36 0)
 			(effects
 				(font
@@
 	(symbol
 		(lib_id "Device:C")
-		(at 102.87 177.8 0)
+		(at 191.77 90.17 0)
 		(unit 1)
 		(exclude_from_sim no)
@@
 		(fields_autoplaced yes)
 		(property "Reference" "C4"
-			(at 106.68 176.5299 0)
+			(at 195.58 88.8999 0)
 			(effects
 				(font
@@
 		)
 		(property "Value" "0.1 uF"
-			(at 106.68 179.0699 0)
+			(at 195.58 91.4399 0)
 			(effects
 				(font
@@
 		)
 		(property "Footprint" "Capacitor_SMD:C_0805_2012Metric"
-			(at 103.8352 181.61 0)
+			(at 192.7352 93.98 0)
 			(effects
 				(font
@@
 		)
 		(property "Datasheet" "~"
-			(at 102.87 177.8 0)
+			(at 191.77 90.17 0)
 			(effects
 				(font
@@
 		)
 		(property "Description" "Unpolarized capacitor"
-			(at 102.87 177.8 0)
+			(at 191.77 90.17 0)
 			(effects
 				(font

Commit message: finished first layout and routing pass
Parts:
- removed TP1, TP10, TP2, TP5, TP6, TP7, TP8, TP9: TestPoint_Probe, TestPoint:TestPoint_Pad_D1.5mm, symbol Connector:TestPoint_Probe
- added C10, C11: 22uF, Capacitor_SMD:C_0805_2012Metric, symbol Device:C
- added C5: 10uF, Capacitor_SMD:C_0805_2012Metric_Pad1.18x1.45mm_HandSolder, symbol Device:C
- added C6, C8: 100nF, Capacitor_SMD:C_0805_2012Metric, symbol Device:C
- added C7: 10uF, Capacitor_SMD:C_0805_2012Metric, symbol Device:C
- added C9: 22pF, Capacitor_SMD:C_0805_2012Metric, symbol Device:C
- added L3: 4.7uH, Inductor_SMD:L_0805_2012Metric_Pad1.15x1.40mm_HandSolder, symbol Device:L
- added R8: 52.3kΩ, Resistor_SMD:R_0805_2012Metric_Pad1.20x1.40mm_HandSolder, symbol Device:R
- added R9: 10kΩ, Resistor_SMD:R_0805_2012Metric_Pad1.20x1.40mm_HandSolder, symbol Device:R
- added U4: TPS562202, Package_TO_SOT_SMD:SOT-563, symbol Regulator_Switching:TPS562202
- R1, R2, R3, R4, R5: footprint Resistor_SMD:R_0805_2012Metric -> Resistor_SMD:R_0805_2012Metric_Pad1.20x1.40mm_HandSolder
Connections:
- net +3.3V is gone; now on net CAN3v3: R6.1, R7.1
- net +12V: now also C5.1, C6.1, U4.1 (VIN), U4.5 (EN)
- net +5V: now also C10.1, C9.1, L3.2, R8.1
- net ABSA: now also U2.24 (17_A3_TX4_SDA1); no longer U2.21 (14_A0_TX3_SPDIF_OUT)
- net CSM1: now also U2.26 (19_A5_SCL0); no longer U2.22 (15_A1_RX3_SPDIF_IN)
- net CSM2: now also U2.27 (20_A6_TX5_LRCLK1); no longer U2.23 (16_A2_RX4_SCL1)
- net DIR1: now also U2.22 (15_A1_RX3_SPDIF_IN); no longer U2.25 (18_A4_SDA0)
- net DIR2: now also U2.30 (23_A9_CRX1_MCLK1); no longer U2.26 (19_A5_SCL0)
- net ENC1A: now also U2.2 (0_RX1_CRX2_CS1); no longer U2.10 (8_TX2_IN1)
- net ENC1B: now also U2.3 (1_TX1_CTX2_MISO1); no longer U2.11 (9_OUT1C)
- net ENC2A: now also U2.6 (4_BCLK2); no longer U2.13 (11_MOSI_CTX1)
- net ENC2B: now also U2.5 (3_LRCLK2); no longer U2.14 (12_MISO_MQSL)
- net ENC2I: now also U2.4 (2_OUT2); no longer U2.12 (10_CS_MQSR)
- net FLTM1: now also U2.25 (18_A4_SDA0); no longer U2.27 (20_A6_TX5_LRCLK1)
- net GND: now also C11.2, C6.2, C7.2, R9.2, U4.3 (GND)
- net LED1: now also U2.7 (5_IN2); no longer U2.8 (6_OUT1D)
- net LED2: now also U2.8 (6_OUT1D); no longer U2.9 (7_RX2_OUT1A)
- net PWM1: now also U2.23 (16_A2_RX4_SCL1); no longer U2.2 (0_RX1_CRX2_CS1)
- net PWM2: now also U2.29 (22_A8_CTX1); no longer U2.3 (1_TX1_CTX2_MISO1)
- net RGBB: now also U2.9 (7_RX2_OUT1A); no longer U2.6 (4_BCLK2)
- net RGBG: now also U2.11 (9_OUT1C); no longer U2.5 (3_LRCLK2)
- net RGBR: now also U2.10 (8_TX2_IN1); no longer U2.4 (2_OUT2)
- net RGBW: now also U2.12 (10_CS_MQSR); no longer U2.7 (5_IN2)
- new net: C9.2, R8.2, R9.1, U4.6 (VFB)
- new net: C8.1, L3.1, U4.2 (SW)
- new net: C8.2, U4.4 (VBST)
- new net: C10.2, C11.1
- new net: C5.2, C7.1
- no-connect marks 34 -> 29
Other:
- moved on the sheet: TP11, TP12, TP13

Commit message: cleaning
Parts:
- removed C10, C11: 22uF, Capacitor_SMD:C_0805_2012Metric, symbol Device:C
- removed C5: 10uF, Capacitor_SMD:C_0805_2012Metric_Pad1.18x1.45mm_HandSolder, symbol Device:C
- removed C6, C8: 100nF, Capacitor_SMD:C_0805_2012Metric, symbol Device:C
- removed C7: 10uF, Capacitor_SMD:C_0805_2012Metric, symbol Device:C
- removed C9: 22pF, Capacitor_SMD:C_0805_2012Metric, symbol Device:C
- removed L3: 4.7uH, Inductor_SMD:L_0805_2012Metric_Pad1.15x1.40mm_HandSolder, symbol Device:L
- removed LED1: 599-2310-427F, footprints:599-2310_DIA, symbol 2024-05-06_00-08-00:599-2310-427F
- removed R9: 10kΩ, Resistor_SMD:R_0805_2012Metric_Pad1.20x1.40mm_HandSolder, symbol Device:R
- removed TP3, TP4: TestPoint_Probe, TestPoint:TestPoint_Pad_D1.5mm, symbol Connector:TestPoint_Probe
- removed U4: TPS562202, Package_TO_SOT_SMD:SOT-563, symbol Regulator_Switching:TPS562202
- C1, C2, C3, C4: footprint Capacitor_SMD:C_0805_2012Metric -> Capacitor_SMD:C_0805_2012Metric_Pad1.18x1.45mm_HandSolder
- D1, D2, D3, D4: footprint GreenLED:LED_CREE_MLXXXX -> LED_SMD:LED_0805_2012Metric_Pad1.15x1.40mm_HandSolder
- R1: value 25 -> 500
- R2: value 5 -> 150
- R3: value 15 -> 50
- R6, R7: value R -> 10k
- R8: value 52.3kΩ -> 50
- U1, U3: value ~ -> G218v17
Connections:
- net +5V: no longer R8.1
- net LED1: now also R3.2; no longer D3.2 (A)
- net LED2: now also R8.2; no longer D4.2 (A)
- net RGBB: no longer names the net of U2.9 (7_RX2_OUT1A)
- net RGBG: no longer names the net of U2.11 (9_OUT1C)
- net RGBR: no longer names the net of R3.1
- net RGBR: now also D3.2 (A); no longer U2.10 (8_TX2_IN1)
- net RGBW: no longer names the net of U2.12 (10_CS_MQSR)
- new net: D4.2 (A), R8.1
- no-connect marks 29 -> 35
Other:
- note added: "This is a guess"
- moved on the sheet: D3, D4

Commit message: finalize pcb
Parts:
- added C10, C7: 0.1uF, Capacitor_SMD:C_0805_2012Metric_Pad1.18x1.45mm_HandSolder, symbol Device:C
- added C5, C6: 22uF, Capacitor_SMD:C_0805_2012Metric_Pad1.18x1.45mm_HandSolder, symbol Device:C
- added C8, C9: 10uF, Capacitor_SMD:C_0805_2012Metric_Pad1.18x1.45mm_HandSolder, symbol Device:C
- added L3: 3.3uH, Inductor_SMD:L_Abracon_ASPI-0630LR, symbol Device:L
- added R12: 10K, Resistor_SMD:R_0805_2012Metric_Pad1.20x1.40mm_HandSolder, symbol Device:R_US
- added R13: 54.9K, Resistor_SMD:R_0805_2012Metric_Pad1.20x1.40mm_HandSolder, symbol Device:R_US
- added U4: TPS565208, Package_TO_SOT_SMD:SOT-23-6, symbol Regulator_Switching:TPS565208
Connections:
- net +12V: now also C10.1, C8.1, C9.1, U4.3 (VIN)
- net +5V: now also C5.1, C6.1, L3.2, R13.2
- net GND: now also C10.2, C5.2, C6.2, C8.2, C9.2, R12.1, U4.1 (GND)
- new net: C7.2, L3.1, U4.2 (SW)
- new net: R12.2, R13.1, U4.4 (VFB)
- new net: C7.1, U4.6 (VBST)
- no-connect marks 35 -> 36
Other:
- note added: "12V to 5V, 3A"
- note added: "Note: EN floating to turn on as soon as it gets power"
