File: mainBoard/mainBoard.kicad_pcb (KiCad board)
At the start: 4 copper layers, 78 parts, among them IC1 TCAN3414DR, J1 XT60PW-M, J10 RJ45, J11 RJ45, J12 Conn_01x03, J13 RJ45, J14 RJ45, J15 RJ45, J16 BM04B-SRSS-TB, J17 BM04B-SRSS-TB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

Commit message: updated capacitor value for can split termination
Parts:
- C16: value 270pF -> 560pF
Changed lines of the file:
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@@
 		(sheetname "Data Stuff")
 		(sheetfile "page2.kicad_sch")
-		(attr smd dnp)
+		(attr smd)
 		(fp_line
 			(start -0.227064 -0.735)
@@
 			)
 		)
-		(property "Value" "270pF"
+		(property "Value" "560pF"
 			(at 0 1.68 90)
 			(layer "F.Fab")
@@
 		(sheetname "Data Stuff")
 		(sheetfile "page2.kicad_sch")
-		(attr smd dnp)
+		(attr smd)
 		(fp_line
 			(start -0.261252 -0.735)
@@
 		(sheetname "Data Stuff")
 		(sheetfile "page2.kicad_sch")
-		(attr smd dnp)
+		(attr smd)
 		(fp_line
 			(start -0.227064 -0.735)

Commit message: Added mainboard step
Other:
- board outline added: 132 x 85 mm
Changed lines of the file:
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@@
 		(pad_to_mask_clearance 0)
 		(allow_soldermask_bridges_in_footprints no)
+		(grid_origin 21 97)
 		(pcbplotparams
 			(layerselection 0x00010fc_ffffffff)
@@
 		)
 	)
+	(gr_rect
+		(start 21 12)
+		(end 153 97)
+		(stroke
+			(width 0.1)
+			(type default)
+		)
+		(fill none)
+		(layer "Edge.Cuts")
+	)
 )
