File: solenoid_driver2.0/solenoid driver 2.0.kicad_pcb (KiCad board)
At the start: 2 copper layers, 32.5 x 54 mm, 12 parts, among them J1 12v and gnd, J2 solenoid1 screw terminal, J3 signal 1 and 2, J4 solenoid2 screw terminal, Q1 IRF3205, Q2 IRF3205

Commit message: updates to manufacture
Routing:
- net pin2: track 17.1 -> 36.2 mm, vias 1 -> 0
- net +12V: track 71.5 -> 79.6 mm, vias 1 -> 0
- net drain1: track 21.7 -> 24.8 mm
- net pin1: track 13.4 -> 14.0 mm, vias 2 -> 0
Other:
- board size 32.5 x 54 mm -> 34.5 x 54 mm
